Commit message: Mejora en los links para eliminar ese desbalance de altura en rviz

File: description2/urdf/robot_rover.gazebo.xacro (robot description, xacro)
@@ -84,5 +84,5 @@
             <odometryTopic>odom</odometryTopic>
             <odometryFrame>odom</odometryFrame>
-            <robotBaseFrame>base_link</robotBaseFrame>
+            <robotBaseFrame>base_footprint</robotBaseFrame>
             <publishWheelTF>false</publishWheelTF>
             <publishTf>true</publishTf>

File: description2/urdf/robot_rover.urdf.xacro (robot description, xacro)
@@ -3,12 +3,11 @@
   <xacro:include filename="$(find description2)/urdf/materials.xacro"/>
   <xacro:include filename="$(find description2)/urdf/robot_rover.gazebo.xacro"/>
-  <link name="base_link">
-  </link>
-  <joint name="chassis_joint" type="fixed">
-    <parent link = "base_link"/>
-    <child link = "chassis"/>
-    <origin xyz ="0 0 0"/>
+  <link name="base_footprint"/>
+  <joint name="main_joint" type="fixed">
+    <parent link = "base_footprint"/>
+    <child link = "base_link"/>
+    <origin xyz ="0 0 0.10" rpy="0 0 0"/>
   </joint>
-  <link name = "chassis">
+  <link name = "base_link">
     <visual>
       <origin xyz= "0 0 0.085"/>
